File: pcb/FloppyOverdrive_ControlBoard.kicad_pcb (KiCad board)
At the start: 2 copper layers, 163 x 104 mm, 58 parts, among them J1 174804-1, J2 Motor_Header, J3 Floppy_Bus, J4 Sensor_Header, J5 Heads_Header, J6 Step_Header, J7 PIC_ADC_Header, J8 FPGA_IO_Header, J9 HeadOut_Header, SW1 RST_Btn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

Commit message: Backup sync
Other:
- board text added: "Replaces Mitsubishi NAMFN motherboard"
- board text removed: "Replaces Mistubishi NAMFN motherboard"
Changed lines of the file:
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@@
   )
   (setup
+    (stackup
+      (layer "F.SilkS" (type "Top Silk Screen"))
+      (layer "F.Paste" (type "Top Solder Paste"))
+      (layer "F.Mask" (type "Top Solder Mask") (thickness 0.01))
+      (layer "F.Cu" (type "copper") (thickness 0.035))
+      (layer "dielectric 1" (type "core") (thickness 1.51) (material "FR4") (epsilon_r 4.5) (loss_tangent 0.02))
+      (layer "B.Cu" (type "copper") (thickness 0.035))
+      (layer "B.Mask" (type "Bottom Solder Mask") (thickness 0.01))
+      (layer "B.Paste" (type "Bottom Solder Paste"))
+      (layer "B.SilkS" (type "Bottom Silk Screen"))
+      (copper_finish "None")
+      (dielectric_constraints no)
+    )
     (pad_to_mask_clearance 0)
     (aux_axis_origin 227 146)
@@
     (effects (font (size 1 1) (thickness 0.15)))
   )
-  (gr_text "Replaces Mistubishi NAMFN motherboard" (at 80.1 144.7) (layer "F.SilkS")
+  (gr_text "Replaces Mitsubishi NAMFN motherboard" (at 80.1 144.7) (layer "F.SilkS")
     (effects (font (size 1 1) (thickness 0.15)))
   )
