File: pcb/FloppyOverdrive_ControlBoard.kicad_pcb (KiCad board)
At the start: 2 copper layers, 163 x 104 mm, 58 parts, among them J1 174804-1, J2 Motor_Header, J3 Floppy_Bus, J4 Sensor_Header, J5 Heads_Header, J6 Step_Header, J7 PIC_ADC_Header, J8 FPGA_IO_Header, J9 HeadOut_Header, SW1 RST_Btn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

Commit message: Added neg voltage and amps
Parts:
- added C8: 47u, Capacitor_THT:C_Disc_D5.0mm_W2.5mm_P2.50mm, F.Cu at (108.1, 100.8)
- added C9: 47u, Capacitor_THT:C_Disc_D5.0mm_W2.5mm_P2.50mm, F.Cu at (121.3, 103.3)
- added IC1: THS4521IDR, MAX660MX⁄NOPB:SOIC127P600X175-8N, F.Cu at (99.9, 111.3)
- added IC2: THS4521IDR, MAX660MX⁄NOPB:SOIC127P600X175-8N, F.Cu at (99.9, 118.1)
- added IC3: MAX660MX_NOPB, MAX660MX⁄NOPB:SOIC127P600X175-8N, F.Cu at (114.2, 102.0)
- added J10: Flop_ADC_Header, Connector_PinHeader_2.54mm:PinHeader_1x02_P2.54mm_Vertical, F.Cu at (98.8, 123.6)
- added JP2: HeadPos_Sel, Connector_PinHeader_2.54mm:PinHeader_1x03_P2.54mm_Vertical, F.Cu at (97.7, 101.2)
- added JP3: HeadNeg_Sel, Connector_PinHeader_2.54mm:PinHeader_1x03_P2.54mm_Vertical, F.Cu at (97.7, 105.9)
- added R16: 10k, Resistor_SMD:R_0402_1005Metric, F.Cu at (94.3, 112.7)
- added R17: 10k, Resistor_SMD:R_0402_1005Metric, F.Cu at (93.9, 118.6)
- added R18: 1k, Resistor_SMD:R_0402_1005Metric, F.Cu at (94.3, 108.9)
- added R19: 1k, Resistor_SMD:R_0402_1005Metric, F.Cu at (105.0, 114.8)
- added R20: 10k, Resistor_SMD:R_0402_1005Metric, F.Cu at (124.7, 101.1)
- added R21: 10k, Resistor_SMD:R_0402_1005Metric, F.Cu at (124.7, 104.2)
- added R22: 1k, Resistor_SMD:R_0402_1005Metric, F.Cu at (94.9, 114.8)
- added R23: 1k, Resistor_SMD:R_0402_1005Metric, F.Cu at (105.1, 108.9)
- added R24: 10k, Resistor_SMD:R_0402_1005Metric, F.Cu at (105.1, 112.7)
- added R25: 10k, Resistor_SMD:R_0402_1005Metric, F.Cu at (105.5, 117.9)
- added TP16: TP_-2V5, TestPoint:TestPoint_Pad_D1.0mm, F.Cu at (128.1, 104.2)
- added TP17: TP_2V5, TestPoint:TestPoint_Pad_D1.0mm, F.Cu at (128.0, 100.3)
Routing:
- net +2V5: track 0.00 -> 57.3 mm, vias 0 -> 3
- net -2V5: track 0.00 -> 46.7 mm, vias 0 -> 4
- net GND: track 65.3 -> 87.1 mm, vias 2 -> 5
- net Start_1: track 12.9 -> 31.4 mm
- net End_1: track 12.7 -> 29.8 mm
- net Net-(IC2-Pad1): track 0.00 -> 13.7 mm, vias 0 -> 2
- net Net-(IC2-Pad8): track 0.00 -> 11.2 mm
- net HeadPos: track 0.00 -> 10.0 mm
- net Start_0: track 12.7 -> 22.6 mm
- net End_0: track 12.7 -> 21.2 mm
- net Neg_Out: track 0.00 -> 8.30 mm
- net Pos_Out: track 0.00 -> 7.93 mm
- net HeadNeg: track 0.00 -> 6.95 mm
- net Net-(IC1-Pad1): track 0.00 -> 5.68 mm
- net Net-(IC1-Pad8): track 0.00 -> 5.28 mm
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Other:
- board text added: "+"
- board text added: "+ -"
- board text added: "+2.5V"
- board text added: "-"
- board text added: "-2.5V"
- board text added: "Amp Out"
- board text added: "Head 0 1"
- board text removed: "FPGA Outputs"
