File: pcb/FloppyOverdrive_ControlBoard.kicad_sch (KiCad schematic)
At the start: 78 parts, among them IC1 THS4521IDR, IC2 THS4521IDR, IC3 MAX660MX_NOPB, J1 174804-1, J10 Flop_ADC_Header, J2 Motor_Header, J3 Floppy_Bus, J4 Sensor_Header, J5 Heads_Header, J6 Step_Header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

Commit message: Fixed pin 39, added missing hole to PCB
Connections:
- net +3.3V is gone; now on net +3V3: J8.39 (Pin_39)
Changed lines of the file:
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@@
     (pin "2")
-  )
-  (symbol (lib_id "power:+3.3V") (at 132.08 135.89 270) (unit 1)
-    (in_bom yes) (on_board yes) (fields_autoplaced)
-    (property "Reference" "#PWR0143" (id 0) (at 128.27 135.89 0)
-      (effects (font (size 1.27 1.27)) hide)
-    )
-    (property "Value" "+3.3V" (id 1) (at 135.89 135.8899 90)
-      (effects (font (size 1.27 1.27)) (justify left))
-    )
-    (property "Footprint" "" (id 2) (at 132.08 135.89 0)
-      (effects (font (size 1.27 1.27)) hide)
-    )
-    (property "Datasheet" "" (id 3) (at 132.08 135.89 0)
-      (effects (font (size 1.27 1.27)) hide)
-    )
-    (pin "1")
   )
   (symbol (lib_id "power:GND") (at 57.15 30.48 90) (unit 1)
@@
     )
     (property "Datasheet" "" (id 3) (at 83.82 39.37 0)
+      (effects (font (size 1.27 1.27)) hide)
+    )
+    (pin "1")
+  )
+  (symbol (lib_id "power:+3V3") (at 132.08 135.89 270) (unit 1)
+    (in_bom yes) (on_board yes) (fields_autoplaced)
+    (property "Reference" "#PWR?" (id 0) (at 128.27 135.89 0)
+      (effects (font (size 1.27 1.27)) hide)
+    )
+    (property "Value" "+3V3" (id 1) (at 135.89 135.8899 90)
+      (effects (font (size 1.27 1.27)) (justify left))
+    )
+    (property "Footprint" "" (id 2) (at 132.08 135.89 0)
+      (effects (font (size 1.27 1.27)) hide)
+    )
+    (property "Datasheet" "" (id 3) (at 132.08 135.89 0)
       (effects (font (size 1.27 1.27)) hide)
     )
@@
       (reference "#PWR0142") (unit 1) (value "GND") (footprint "")
     )
-    (path "/a2873c1c-cb87-4107-9403-ce51b7c7f612"
-      (reference "#PWR0143") (unit 1) (value "+3.3V") (footprint "")
-    )
     (path "/5bcb75a0-9c55-4a33-8423-f203bb16e369"
       (reference "#PWR0144") (unit 1) (value "GND") (footprint "")
@@
       (reference "#PWR0149") (unit 1) (value "-2V5") (footprint "")
     )
+    (path "/b416378d-c8ad-49d0-a119-a8fb20b47699"
+      (reference "#PWR?") (unit 1) (value "+3V3") (footprint "")
+    )
     (path "/37e11e99-5758-4ece-9696-6584471c5ab7"
